File: HW_pulsecal/power.kicad_sch (KiCad schematic)
At the start: 13 parts, among them U3 SGM3204, U4 TX4310

Commit message: update
Parts:
- added C26, C27: 106/16V, Capacitor_SMD:C_0603_1608Metric, symbol Device:C
- added C28, C29: 104/50V, Capacitor_SMD:C_0402_1005Metric, symbol Device:C
- added D5: B5819W, Diode_SMD:D_SOD-123, symbol Device:D
- added J2: USB_C_Receptacle_USB2.0, Connector_USB:USB_C_Receptacle_HRO_TYPE-C-31-M-12, symbol Connector:USB_C_Receptacle_USB2.0
- added J3: Conn_01x02, Connector_JST:JST_PH_S2B-PH-SM4-TB_1x02-1MP_P2.00mm_Horizontal, symbol Connector_Generic_MountingPin:Conn_01x02_MountingPin
- added Q1: AO3401A, Package_TO_SOT_SMD:SOT-23, symbol Transistor_FET:AO3401A
- added R31: 1K, Resistor_SMD:R_0402_1005Metric, symbol Device:R
- added R32, R36: 200K, Resistor_SMD:R_0402_1005Metric, symbol Device:R
- added R33: 10K, Resistor_SMD:R_0402_1005Metric, symbol Device:R
- added R34, R35: 5K1, Resistor_SMD:R_0402_1005Metric, symbol Device:R
- C10, C12: value 106/6.3V -> 106/16V; footprint Capacitor_SMD:C_0402_1005Metric -> Capacitor_SMD:C_0603_1608Metric
- C14, C6, C9: footprint Capacitor_SMD:C_0402_1005Metric -> Capacitor_SMD:C_0603_1608Metric
Connections:
- net GND: now also C26.2, C27.2, C28.2, C29.2, J2.A1 (GND), J2.A12 (GND), J2.B1 (GND), J2.B12 (GND), J2.S1 (SHIELD), J3.2 (Pin_2), J3.MP (MountPin), R33.1, R34.1, R35.1, R36.1
- net VBUS: now also D5.1 (K), Q1.2 (S)
- new net: C28.1, Q1.1 (G), R31.1, R33.2
- new net: J2.B5 (CC2), R35.2
- new net: J2.A5 (CC1), R34.2
- new net +5V: C27.1, D5.2 (A), J2.A4 (VBUS), J2.A9 (VBUS), J2.B4 (VBUS), J2.B9 (VBUS), R31.2
- new net +BATT: C26.1, J3.1 (Pin_1), Q1.3 (D), R32.2
- new net bat_adc: C29.1, R32.1, R36.2
- no-connect marks 0 -> 6
Other:
- note added: "PORT"
- moved on the sheet: C6

Commit message: update
Parts:
- R34, R35: value 5K1 -> 5.1K
- U4: value TX4310 -> TX4310B
Changed lines of the file:
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@@
 			)
 		)
-		(property "Value" "5K1"
+		(property "Value" "5.1K"
 			(at 137.16 116.84 90)
 			(effects
@@
 		(on_board yes)
 		(dnp no)
-		(fields_autoplaced yes)
 		(property "Reference" "U3"
-			(at 107.315 67.31 0)
+			(at 107.442 68.326 0)
 			(effects
 				(font
@@
 		)
 		(property "Value" "SGM3204"
-			(at 107.315 69.85 0)
+			(at 107.442 70.866 0)
 			(effects
 				(font
@@
 			)
 		)
-		(property "Value" "5K1"
+		(property "Value" "5.1K"
 			(at 137.16 114.3 90)
 			(effects
@@
 			)
 		)
-		(property "Value" "TX4310"
+		(property "Value" "TX4310B"
 			(at 78.105 27.94 0)
 			(effects

Commit message: update
Other:
- note added: "负压产生"
- company: (none) -> 模拟龙仪器仪表
- title: (none) -> 率表/定标器测试工具
- moved on the sheet: C26, C28, D5, Q1, R31, R33
