File: HW_pulsecal/disp.kicad_sch (KiCad schematic)
At the start: 28 parts, among them SW1 SW_Push, SW10 SW_Push, SW11 SW_Push, SW2 SW_Push, SW3 SW_Push, SW4 SW_Push, SW5 SW_Push, SW6 SW_Push, SW7 SW_Push, SW8 SW_Push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

Commit message: update
Parts:
- removed D3: GS2040AR, Display_7Segment:CA56-12EWA, symbol Display_Character:CC56-12EWA
- removed D4, D5, D6, D7: LED, symbol Device:LED
- removed SW11, SW5, SW8, SW9: SW_Push, symbol Switch:SW_Push
- added D3: display-led-0.39in-6dig, NewLib:display-led-0.39in-6dig, symbol NewLib:display-led-0.39in-6dig
- added R28, R29, R30: 10K, Resistor_SMD:R_0402_1005Metric, symbol Device:R
- R16, R17, R18, R19, R20, R21, R22, R23, R24, R25, R26, R27: footprint (none) -> Resistor_SMD:R_0402_1005Metric
- SW1, SW2, SW3, SW4: footprint (none) -> Button_Switch_SMD:SW_SPST_PTS647_Sx38
- SW5: renamed from SW6; footprint (none) -> Button_Switch_SMD:SW_SPST_PTS647_Sx38
- SW6: renamed from SW7; footprint (none) -> Button_Switch_SMD:SW_SPST_PTS647_Sx38
- SW7: renamed from SW10; footprint (none) -> Button_Switch_SMD:SW_SPST_PTS647_Sx38
Connections:
- net GND: now also SW1.2, SW2.2, SW3.2, SW4.2, SW5.2, SW6.2, SW7.2
- net at R26.2: now also D3.13 (K)
- net key_freq: now reaches SW2.1
- net key_volt: now reaches SW3.1
- net at R25.2: now also D3.21 (J)
- net at R20.2: now also D3.6 (E)
- net at R21.2: now also D3.19 (F)
- net at R16.2: now also D3.18 (A)
- net at R19.2: now also D3.4 (D)
- net at R23.2: now also D3.10 (G2)
- net at R18.2: now also D3.3 (C)
- net at R22.2: now also D3.11 (G1)
- net at R17.2: now also D3.16 (B)
- net key_move: now reaches SW6.1
- net at R24.2: now also D3.22 (H)
- net at R27.2: now also D3.9 (L)
- net key_pulse: now reaches SW1.1
- net key_add: now reaches SW5.1
- net key_output: now reaches SW4.1
- net key_sub: now reaches SW7.1
- net DIG_a renamed DISP_A
- net DIG_b renamed DISP_B
- net DIG_c renamed DISP_C
- net DIG_d renamed DISP_D
- net DIG_dp renamed DISP_G2
- net DIG_e renamed DISP_E
- net DIG_f renamed DISP_F
- net DIG_g renamed DISP_G1
- net led_hv renamed DISP_H
- net led_hz renamed DISP_K
- net led_ns renamed DISP_J
- net led_volt renamed DISP_L
- new net: D3.8 (M), R28.2
- new net: D3.5 (DP), R30.2
- new net: D3.7 (N), R29.2
- new net DISP_DIG1: D3.2 (DIG1)
- new net DISP_DIG2: D3.20 (DIG2)
- new net DISP_DIG3: D3.17 (DIG3)
- new net DISP_DIG4: D3.15 (DIG4)
- new net DISP_DIG5: D3.14 (DIG5)
- new net DISP_DIG6: D3.12 (DIG6)
- new net DISP_DP: R30.1
- new net DISP_M: R28.1
- new net DISP_N: R29.1
Other:
- note added: "+1"
- note added: "-1"
- note added: "0.1~5000000"
- note added: "50~9999"
- note added: "5~1000"
- note added: "Hz/KHz/MHz"
- note added: "output"
- note added: "按下设置相应的设置项，有些按两次切换单位"
- note added: "换位"
- moved on the sheet: SW1, SW2, SW3, SW5, SW6, SW7

Commit message: update
Parts:
- R16, R17, R18, R19, R20, R21, R22, R23, R24, R25, R26, R27, R28, R29, R30: value 10K -> 330R
- SW1, SW2, SW3, SW4, SW5, SW6, SW7: value SW_Push -> 6*6*5 100g; footprint Button_Switch_SMD:SW_SPST_PTS647_Sx38 -> Button_Switch_SMD:SW_SPST_PTS645
Changed lines of the file:
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@@
 			)
 		)
-		(property "Value" "10K"
+		(property "Value" "330R"
 			(at 48.26 30.48 90)
 			(effects
@@
 			)
 		)
-		(property "Value" "SW_Push"
+		(property "Value" "6*6*5 100g"
 			(at 48.26 101.6 0)
 			(effects
@@
 			)
 		)
-		(property "Footprint" "Button_Switch_SMD:SW_SPST_PTS647_Sx38"
+		(property "Footprint" "Button_Switch_SMD:SW_SPST_PTS645"
 			(at 48.26 101.6 0)
 			(effects
@@
 			)
 		)
-		(property "Value" "SW_Push"
+		(property "Value" "6*6*5 100g"
 			(at 48.26 114.3 0)
 			(effects
@@
 			)
 		)
-		(property "Footprint" "Button_Switch_SMD:SW_SPST_PTS647_Sx38"
+		(property "Footprint" "Button_Switch_SMD:SW_SPST_PTS645"
 			(at 48.26 114.3 0)
 			(effects
@@
 			)
 		)
-		(property "Value" "10K"
+		(property "Value" "330R"
 			(at 48.26 58.42 90)
 			(effects
@@
 			)
 		)
-		(property "Value" "10K"
+		(property "Value" "330R"
 			(at 48.26 40.64 90)
 			(effects
@@
 			)
 		)
-		(property "Value" "10K"
+		(property "Value" "330R"
 			(at 48.26 63.5 90)
 			(effects
@@
 			)
 		)
-		(property "Value" "10K"
+		(property "Value" "330R"
 			(at 48.26 27.94 90)
 			(effects
@@
 			)
 		)
-		(property "Value" "10K"
+		(property "Value" "330R"
 			(at 48.26 55.88 90)
 			(effects
@@
 			)
 		)
-		(property "Value" "SW_Push"
+		(property "Value" "6*6*5 100g"
 			(at 73.66 101.6 0)
 			(effects
@@
 			)
 		)
-		(property "Footprint" "Button_Switch_SMD:SW_SPST_PTS647_Sx38"
+		(property "Footprint" "Button_Switch_SMD:SW_SPST_PTS645"
 			(at 73.66 101.6 0)
 			(effects
@@
 			)
 		)
-		(property "Value" "10K"
+		(property "Value" "330R"
 			(at 48.26 35.56 90)
 			(effects
@@
 			)
 		)
-		(property "Value" "10K"
+		(property "Value" "330R"
 			(at 48.26 60.96 90)
 			(effects
@@
 			)
 		)
-		(property "Value" "SW_Push"
+		(property "Value" "6*6*5 100g"
 			(at 48.26 127 0)
 			(effects
@@
 			)
 		)
-		(property "Footprint" "Button_Switch_SMD:SW_SPST_PTS647_Sx38"
+		(property "Footprint" "Button_Switch_SMD:SW_SPST_PTS645"
 			(at 48.26 127 0)
 			(effects
@@
 			)
 		)
-		(property "Value" "SW_Push"
+		(property "Value" "6*6*5 100g"
 			(at 48.26 88.9 0)
 			(effects
@@
 			)
 		)
-		(property "Footprint" "Button_Switch_SMD:SW_SPST_PTS647_Sx38"
+		(property "Footprint" "Button_Switch_SMD:SW_SPST_PTS645"
 			(at 48.26 88.9 0)
 			(effects
@@
 			)
 		)
-		(property "Value" "SW_Push"
+		(property "Value" "6*6*5 100g"
 			(at 73.66 88.9 0)
 			(effects
@@
 			)
 		)
-		(property "Footprint" "Button_Switch_SMD:SW_SPST_PTS647_Sx38"
+		(property "Footprint" "Button_Switch_SMD:SW_SPST_PTS645"
 			(at 73.66 88.9 0)
 			(effects
@@
 			)
 		)
-		(property "Value" "10K"
+		(property "Value" "330R"
 			(at 48.26 45.72 90)
 			(effects
@@
 			)
 		)
-		(property "Value" "10K"
+		(property "Value" "330R"
 			(at 48.26 48.26 90)
 			(effects
@@
 			)
 		)
-		(property "Value" "10K"
+		(property "Value" "330R"
 			(at 48.26 50.8 90)
 			(effects
@@
 			)
 		)
-		(property "Value" "10K"
+		(property "Value" "330R"
 			(at 48.26 38.1 90)
 			(effects
@@
 			)
 		)
-		(property "Value" "SW_Push"
+		(property "Value" "6*6*5 100g"
 			(at 73.66 114.3 0)
 			(effects
@@
 			)
 		)
-		(property "Footprint" "Button_Switch_SMD:SW_SPST_PTS647_Sx38"
+		(property "Footprint" "Button_Switch_SMD:SW_SPST_PTS645"
 			(at 73.66 114.3 0)
 			(effects
@@
 			)
 		)
-		(property "Value" "10K"
+		(property "Value" "330R"
 			(at 48.26 43.18 90)
 			(effects
@@
 			)
 		)
-		(property "Value" "10K"
+		(property "Value" "330R"
 			(at 48.26 53.34 90)
 			(effects
@@
 			)
 		)
-		(property "Value" "10K"
+		(property "Value" "330R"
 			(at 48.26 33.02 90)
 			(effects

Commit message: update
Other:
- company: (none) -> 模拟龙仪器仪表
- title: (none) -> 率表/定标器测试工具
- moved on the sheet: D3, R16, R17, R18, R19, R20, R21, R22, R23, R24, R25, R26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

Commit message: UPDATE
改连接器和输入电路
Other:
- note added: "move"
- note removed: "按下设置相应的设置项，有些按两次切换单位"
- note removed: "换位"
Changed lines of the file:
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@@
 	(rectangle
 		(start 20.32 83.82)
-		(end 115.57 162.56)
+		(end 115.57 151.13)
 		(stroke
 			(width 0)
@@
 		)
 	)
-	(text "按下设置相应的设置项，有些按两次切换单位\n"
-		(exclude_from_sim no)
-		(at 31.242 145.542 0)
-		(effects
-			(font
-				(size 1.27 1.27)
-			)
-			(justify left top)
-		)
-	)
 	(text "-1"
 		(exclude_from_sim no)
@@
 		)
 	)
-	(text "换位"
+	(text "move"
 		(exclude_from_sim no)
 		(at 83.82 113.792 0)
