File: HW_pulsecal/pulsecal.kicad_pcb (KiCad board)
At the start: 2 copper layers, 98 x 98 mm, 95 parts, among them J1 BNC_CONN, J2 USB_C_Receptacle_USB2.0, J3 Conn_01x02, J4 Conn_01x04, Q1 AO3401A, Q3 FDG6301N, SW1 6*6*5 100g, SW2 6*6*5 100g, SW3 6*6*5 100g, SW4 6*6*5 100g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

Commit message: update
Parts:
- added D4: BSD3A031LV45, Diode_SMD:D_SOD-323_HandSoldering, F.Cu at (44.9, 70.3)
- D1: value SMBJ3.3CA -> BSD3A031LV45; footprint Diode_SMD:D_SMB -> Diode_SMD:D_SOD-323_HandSoldering
- moved D1 6.28 mm to (49.2, 69.1), turned to 0 degrees
- moved Q3 2.78 mm to (48.6, 72.4)
- moved R37 2.78 mm to (51.1, 73.0)
- moved C2 2.77 mm to (53.0, 73.0)
- moved C20 1.95 mm to (46.0, 76.7)
- moved C21 1.95 mm to (50.1, 76.7)
- moved R8 1.95 mm to (47.1, 76.7)
- moved R9 1.95 mm to (49.0, 76.7)
Connections:
- D1 pad 1: GND -> Net-(D1-A1)
- D1 pad 2: Net-(D1-A2) -> GND
- Q3 pad 1: Net-(D1-A2) -> Net-(D1-A1)
- Q3 pad 3: Net-(D1-A2) -> Net-(D1-A1)
- R1 pad 2: Net-(D1-A2) -> Net-(D1-A1)
Routing:
- net Net-(D1-A1): track 0.00 -> 22.8 mm
- net Net-(D1-A2): track 17.7 -> 0.00 mm
- net GND: track 142.3 -> 147.1 mm, vias 449 -> 451
- net Net-(Q3A-D): track 8.86 -> 11.2 mm
- net pulse: track 12.9 -> 10.9 mm
- net pulse_n: track 10.0 -> 8.09 mm
- net Net-(Q3A-G): track 7.79 -> 6.97 mm
- net Net-(Q3B-G): track 4.87 -> 4.04 mm

Commit message: update
Parts:
- removed D4: BSD3A031LV45, Diode_SMD:D_SOD-323_HandSoldering
- added R12: 1R, Resistor_SMD:R_0402_1005Metric, F.Cu at (48.0, 76.7)
- C2: value NC -> 105/25V
- D1: value BSD3A031LV45 -> SMBJ3.3A; footprint Diode_SMD:D_SOD-323_HandSoldering -> Diode_SMD:D_SMB
- J1: value BNC_CONN -> MHV-KE
- R11: value 2.2K -> 22K
- R15: value 1K -> 10K
- moved D1 6.89 mm to (42.7, 71.3), turned to -90 degrees
- moved C20 0.75 mm to (45.2, 76.7)
- moved R8 0.75 mm to (46.4, 76.7)
- moved C21 0.55 mm to (50.6, 76.7)
- moved R9 0.55 mm to (49.5, 76.7)
Connections:
- Q3 pad 4: GND -> Net-(Q3B-S)
Routing:
- net GND: track 147.1 -> 141.7 mm, vias 451 -> 455
- net Net-(Q3B-S): track 0.00 -> 2.77 mm
- net Net-(Q3A-G): track 6.97 -> 7.59 mm
- net pulse_n: track 8.09 -> 7.48 mm
Other:
- board text added: "V1.2a"
- board text removed: "V1.2"
